File: hardware/kicad/b2500_cluster_pwm_dimmer.kicad_pcb (KiCad board)
At the start: 2 copper layers, 94 x 62 mm, 36 parts, among them J1 Phoenix MKDS-1,5-5-5.08, Q1 FQP27P06, Q2 2N7000, SW1 CAL, U1 XIAO RP2040, U2 Pololu D36V28F5

Commit message: Fully route the PCB and export fabrication gerbers
Replace the place-and-pour-only board with a complete, DRC-clean layout
(0 violations, 0 unconnected). gen_pcb.py now includes a self-contained
collision-aware router:

- 2-segment L and 3-segment swept-dogleg attempts on either copper layer,
  with a via dropped at the corner when the legs change layer; rejects any
  candidate within clearance of a foreign pad, track, or via.
- A grid maze (Lee) fallback that guarantees a path where one exists, used
  for the nets boxed in by the XIAO pin columns and the power spines
  (e.g. 3V3, DIM_IN). Grid-discretisation safety margin keeps maze routes
  off pad/track edges.
- High-current nets (VIN_RAW, PWM_OUT, VIN_PROT) at 1.5 mm, signals 0.4 mm.
  VIN_PROT is now routed by the same router instead of a hand trunk.
- Bonds the tactile switch's duplicate same-net legs with copper.

export_fab.py run produces gerbers + Excellon drill in hardware/gerbers/
(ready to manufacture) and refreshes the BOM. README and fabrication_notes
updated: the board is fully routed; no GUI step is required to order it.

Co-Authored-By: Claude Fable 5 <noreply@anthropic.com>
Routing:
- net VIN_PROT: track 0.00 -> 129.0 mm
- net 3V3: track 0.00 -> 55.4 mm
- net IGN_SENSE_RAW: track 0.00 -> 43.3 mm
- net 5V_XIAO: track 0.00 -> 40.7 mm
- net PWM_GATE: track 0.00 -> 37.6 mm, vias 0 -> 2
- net IGN_DIV: track 0.00 -> 37.4 mm
- net CAL_BTN: track 0.00 -> 31.1 mm
- net DIM_ADC: track 0.00 -> 30.7 mm, vias 0 -> 1
- net DIM_IN: track 0.00 -> 29.2 mm, vias 0 -> 2
- net Q1_G: track 0.00 -> 28.2 mm
- net DIM_DIV: track 0.00 -> 23.0 mm
- net Q2_G: track 0.00 -> 20.5 mm
- net Q2_D: track 0.00 -> 16.1 mm
- net 5V_BUCK: track 0.00 -> 14.8 mm
- net 5V_JMP: track 0.00 -> 7.38 mm
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
Commit message: Fix U2 buck land: off-board 3-pin wired header (audit finding)
A datasheet/footprint audit found the U2 land was wrong: the custom Pololu
D36V28F5 footprint had 4 pads in an unverified order, but the real module has
6 connections (offset PG plus two GNDs) and Pololu does not publish the edge
pin order in text. A mis-built buck could put 12 V on the 5 V rail.

Replace it with an orientation-proof connection: U2 is now a labeled 3-pin
header (VIN / GND / VOUT 5V) for the module mounted off-board and wired
label-to-label. EN (default-on) and PG are unused.

- netlist.py: U2 -> PinHeader_1x03, pads VIN/GND/VOUT -> VIN_PROT/GND/5V_BUCK.
- gen_sch.py: buck symbol reduced to 3 pins (VIN/GND/VOUT). ERC clean.
- gen_pcb.py: re-place U2, add per-pin silk and OFF-BOARD BUCK label, fix the
  VIN_PROT and 5V_BUCK routing pad refs. Fully routed, DRC 0/0.
- Delete the incorrect Pololu_D36V28F5.kicad_mod; refresh gerbers, BOM, docs.

Audit also verified (correct, no change): XIAO RP2040 footprint pinout plus
0.6in/0.1in spacing, FQP27P06 G-D-S, 2N7000 S-G-D, BAT54S pin-3 common, and
diode (cathode = pad 1) polarities.

Co-Authored-By: Claude Fable 5 <noreply@anthropic.com>
Parts:
- U2: value Pololu D36V28F5 -> Pololu D36V28F5 (off-board, wired); footprint Pololu_D36V28F5 -> PinHeader_1x03_P2.54mm_Vertical
- moved U2 2.24 mm to (74.0, 12.0)
Connections:
- U2 pad 1: (no net) -> VIN_PROT
- U2 pad 2: VIN_PROT -> GND
- U2 pad 3: GND -> 5V_BUCK
Routing:
- net 5V_BUCK: track 14.8 -> 22.9 mm
- net VIN_PROT: track 129.0 -> 120.9 mm
Other:
- board text added: "OFF-BOARD BUCK"
- board text added: "VIN"
- board text added: "VOUT 5V"

Commit message: Add green power-on LED (D6 + R11) on protected 12V input
Lights whenever the board has power. 3mm THT green LED with a 3.3k
series resistor (~3 mA) off VIN_PROT, placed top-right with a PWR silk
label. Schematic gains an LED symbol; fully routed, DRC 0/0; gerbers,
BOM, schematic PDF, and render refreshed.

Co-Authored-By: Claude Opus 4.8 <noreply@anthropic.com>
Parts:
- added D6: Green LED (PWR), LED_D3.0mm, F.Cu at (78.0, 20.0)
- added R11: 3.3k, R_0805_2012Metric_Pad1.20x1.40mm_HandSolder, F.Cu at (70.0, 20.0)
Routing:
- net VIN_PROT: track 120.9 -> 133.9 mm
- net LED_A: track 0.00 -> 9.54 mm, vias 0 -> 1
Other:
- board text added: "PWR"
